Commit message: fix gripper in gazebo

File: src/probot_description/urdf/probot.ros2_control.xacro (robot description, xacro)
@@ -66,4 +66,11 @@
                 </state_interface>
             </joint>
+            <xacro:if value="${use_gazebo}">
+                <joint name="Passive_Gear_Joint">
+                    <param name="mimic">Active_Gear_Joint</param>
+                    <param name="multiplier">-1.0</param>
+                    <state_interface name="position"/>
+                </joint>
+            </xacro:if>
             <gpio name="iris_shutter">
                 <command_interface name="state"/>

Commit message: gazebo hot fix and vision

File: src/probot_description/urdf/probot.ros2_control.xacro (robot description, xacro)
@@ -73,5 +73,5 @@
             </joint>
             <xacro:if value="${use_gazebo}">
-                <joint name="Passive_Gear_Joint">
+                <joint name="Passive_Scissors_Gear_Joint">
                     <param name="mimic">Active_Gear_Joint</param>
                     <param name="multiplier">-1.0</param>
