Commit message: add cameras to gazebo

File: src/probot_description/urdf/gripper_macro.xacro (robot description, xacro)
@@ -1,5 +1,5 @@
 <?xml version="1.0"?>
 <robot xmlns:xacro="http://ros.org/wiki/xacro">
-  <xacro:macro name="probot_gripper" params="parent">
+  <xacro:macro name="probot_gripper" params="parent use_gazebo">
     <!-- Standardized Gripper Materials -->
     <material name="gripper_white">
@@ -298,4 +298,53 @@
       <child link="LED2_Link" />
     </joint>
+    <!-- ========================================================= -->
+    <!-- GAZEBO SENSORS: ESP CAMS                                  -->
+    <!-- ========================================================= -->
+    <xacro:if value="${use_gazebo}">
+      <!-- ESP Camera 1 -->
+      <gazebo reference="esp_camera1">
+        <sensor name="esp_camera1_rgb" type="camera">
+          <pose>0 0 0.01 -1.5708 -1.5708 0</pose>
+          <always_on>true</always_on>
+          <update_rate>30.0</update_rate>
+          <visualize>true</visualize>
+          <topic>/camera/esp1/image_raw</topic>
+          <camera>
+            <horizontal_fov>1.047</horizontal_fov>
+            <image>
+              <width>600</width>
+              <height>800</height>
+              <format>R8G8B8</format>
+            </image>
+            <clip>
+              <near>0.01</near>
+              <far>10.0</far>
+            </clip>
+          </camera>
+        </sensor>
+      </gazebo>
+      <!-- ESP Camera 2 -->
+      <gazebo reference="esp_camera2">
+        <sensor name="esp_camera2_rgb" type="camera">
+          <pose>0 0 0.01 -1.5708 -1.5708 0</pose>
+          <always_on>true</always_on>
+          <update_rate>30.0</update_rate>
+          <visualize>true</visualize>
+          <topic>/camera/esp2/image_raw</topic>
+          <camera>
+            <horizontal_fov>1.047</horizontal_fov>
+            <image>
+              <width>600</width>
+              <height>800</height>
+              <format>R8G8B8</format>
+            </image>
+            <clip>
+              <near>0.01</near>
+              <far>10.0</far>
+            </clip>
+          </camera>
+        </sensor>
+      </gazebo>
+    </xacro:if>
   </xacro:macro>
 </robot>

File: src/probot_description/urdf/probot_anno.xacro (robot description, xacro)
@@ -9,6 +9,6 @@
     <xacro:include filename="$(find probot_description)/urdf/gripper_macro.xacro" />
     <xacro:include filename="$(find probot_description)/urdf/probot.ros2_control.xacro" />
-    <xacro:probot_anno_macro />
-    <xacro:probot_gripper parent="link_6" />
+    <xacro:probot_anno_macro use_gazebo="$(arg use_gazebo)" />
+    <xacro:probot_gripper parent="link_6" use_gazebo="$(arg use_gazebo)" />
     <xacro:probot_anno_ros2_control
         name="ProbotSystem"

File: src/probot_description/urdf/probot_anno_macro.xacro (robot description, xacro)
@@ -1,5 +1,5 @@
 <?xml version="1.0"?>
 <robot xmlns:xacro="http://ros.org/wiki/xacro">
-  <xacro:macro name="probot_anno_macro">
+  <xacro:macro name="probot_anno_macro" params="use_gazebo">
     <xacro:property name="M_PI" value="3.1415926536"/>
     <!-- Materials -->
@@ -270,4 +270,30 @@
       <child link="tool0" />
     </joint-->
+    <!-- ========================================================= -->
+    <!-- GAZEBO SENSORS: KINECT RGB-D                              -->
+    <!-- ========================================================= -->
+    <xacro:if value="${use_gazebo}">
+      <gazebo reference="camera_link2">
+        <sensor name="kinect_rgbd" type="rgbd_camera">
+          <pose>0 0 0.01 1.5708 -1.5708 0</pose>
+          <always_on>true</always_on>
+          <update_rate>30.0</update_rate>
+          <visualize>true</visualize>
+          <topic>/camera/kinect</topic>
+          <camera>
+            <horizontal_fov>1.047</horizontal_fov>
+            <image>
+              <width>640</width>
+              <height>480</height>
+              <format>R8G8B8</format>
+            </image>
+            <clip>
+              <near>0.05</near>
+              <far>10.0</far>
+            </clip>
+          </camera>
+        </sensor>
+      </gazebo>
+    </xacro:if>
     </xacro:macro>
 </robot>

Commit message: add target frame

File: src/probot_description/urdf/gripper_macro.xacro (robot description, xacro)
@@ -297,4 +297,11 @@
       <parent link="Container_link" />
       <child link="LED2_Link" />
+    </joint>
+    <!-- Grasp target frame -->
+    <link name="grasp_target_link" />
+    <joint name="grasp_target_joint" type="fixed">
+      <origin xyz="0 0 0.1035" rpy="0 0 0" />
+      <parent link="Container_link" />
+      <child link="grasp_target_link" />
     </joint>
     <!-- ========================================================= -->
