Commit message: add gazebo package

File: src/probot_description/urdf/probot_anno_macro.xacro (robot description, xacro)
@@ -3,8 +3,8 @@
   <xacro:macro name="probot_anno_macro">
     <xacro:property name="M_PI" value="3.1415926536"/>
-    <link name="base_footprint"/>
+    <link name="world"/>
     <joint name="joint_0" type="fixed">
       <origin xyz="0 0 0.0532" rpy="0 0 0" />
-      <parent link="base_footprint" />
+      <parent link="world" />
       <child link="base_link" />
     </joint>

Commit message: autonomous 101

File: src/probot_description/urdf/probot_anno_macro.xacro (robot description, xacro)
@@ -47,5 +47,6 @@
     <link name="camera_link2"/>
     <joint name="camera_joint2" type="fixed">
-      <origin xyz="-0.32393 0.13681 0.05339" rpy="-1.509 0 0" />
+      <!-- <origin xyz="-0.32393 0.13681 0.05339" rpy="-1.509 0 0" /> -->
+      <origin xyz="-0.32393 0.13681 0.05339" rpy="-0.7236 0 0" />
       <parent link="robot_base" />
       <child link="camera_link2" />
@@ -276,4 +277,5 @@
       <gazebo reference="camera_link2">
         <sensor name="kinect_rgbd" type="rgbd_camera">
+          <gz_frame_id>camera_link2</gz_frame_id>
           <pose>0 0 0.01 1.5708 -1.5708 0</pose>
           <always_on>true</always_on>
