Commit message: gazebo and hardware integration

File: src/moveit_config/config/probot_anno.urdf.xacro (robot description, xacro)
@@ -1,9 +1,4 @@
 <?xml version="1.0"?>
 <robot xmlns:xacro="http://www.ros.org/wiki/xacro" name="probot_anno">
-    <xacro:arg name="initial_positions_file" default="initial_positions.yaml" />
-    <!-- Import probot_anno urdf file -->
     <xacro:include filename="$(find probot_description)/urdf/probot_anno.xacro" />
-    <!-- Import control_xacro -->
-    <xacro:include filename="probot_anno.ros2_control.xacro" />
-    <xacro:probot_anno_ros2_control name="FakeSystem" initial_positions_file="$(arg initial_positions_file)"/>
 </robot>

File: src/probot_description/urdf/probot.ros2_control.xacro (robot description, xacro)
@@ -1,50 +1,64 @@
 <?xml version="1.0"?>
 <robot xmlns:xacro="http://www.ros.org/wiki/xacro">
-  <xacro:macro name="probot_ros2_control" params="name">
-    <ros2_control name="${name}" type="system">
-      <hardware>
-        <plugin>gz_ros2_control/GazeboSimSystem</plugin>
-      </hardware>
-      <joint name="joint_1">
-        <command_interface name="position"/>
-        <state_interface name="position"><param name="initial_value">0.0</param></state_interface>
-        <state_interface name="velocity"/>
-      </joint>
-      <joint name="joint_2">
-        <command_interface name="position"/>
-        <state_interface name="position"><param name="initial_value">0.0</param></state_interface>
-        <state_interface name="velocity"/>
-      </joint>
-      <joint name="joint_3">
-        <command_interface name="position"/>
-        <state_interface name="position"><param name="initial_value">0.0</param></state_interface>
-        <state_interface name="velocity"/>
-      </joint>
-      <joint name="joint_4">
-        <command_interface name="position"/>
-        <state_interface name="position"><param name="initial_value">0.0</param></state_interface>
-        <state_interface name="velocity"/>
-      </joint>
-      <joint name="joint_5">
-        <command_interface name="position"/>
-        <state_interface name="position"><param name="initial_value">0.0</param></state_interface>
-        <state_interface name="velocity"/>
-      </joint>
-      <joint name="joint_6">
-        <command_interface name="position"/>
-        <state_interface name="position"><param name="initial_value">0.0</param></state_interface>
-        <state_interface name="velocity"/>
-      </joint>
-      <!--joint name="finger_joint1">
-        <command_interface name="position" />
-        <state_interface name="position" />
-        <state_interface name="velocity" />
-      </joint-->
-    </ros2_control>
-    <gazebo>
-      <plugin filename="gz_ros2_control-system" name="gz_ros2_control::GazeboSimROS2ControlPlugin">
-        <parameters>$(find moveit_config)/config/ros2_controllers.yaml</parameters>
-      </plugin>
-    </gazebo>
-  </xacro:macro>
+    <xacro:macro name="probot_anno_ros2_control" params="name initial_positions_file use_mock_hardware use_real_hardware use_gazebo use_isaac">
+        <xacro:property name="initial_positions" value="${load_yaml(initial_positions_file)['initial_positions']}"/>
+        <ros2_control name="${name}" type="system">
+            <hardware>
+                <xacro:if value="${use_mock_hardware}">
+                    <plugin>mock_components/GenericSystem</plugin>
+                </xacro:if>
+                <xacro:if value="${use_real_hardware}">
+                    <plugin>probot_hardware/ProbotSystemHardware</plugin>
+                </xacro:if>
+                <xacro:if value="${use_gazebo}">
+                    <plugin>ign_ros2_control/IgnitionSystem</plugin>
+                </xacro:if>
+                <xacro:if value="${use_isaac}">
+                    <plugin>topic_based_ros2_control/TopicBasedSystem</plugin>
+                </xacro:if>
+            </hardware>
+            <joint name="joint_1">
+                <command_interface name="position"/>
+                <state_interface name="position">
+                  <param name="initial_value">${initial_positions['joint_1']}</param>
+                </state_interface>
+                <!--state_interface name="velocity"/-->
+            </joint>
+            <joint name="joint_2">
+                <command_interface name="position"/>
+                <state_interface name="position">
+                  <param name="initial_value">${initial_positions['joint_2']}</param>
+                </state_interface>
+                <!--state_interface name="velocity"/-->
+            </joint>
+            <joint name="joint_3">
+                <command_interface name="position"/>
+                <state_interface name="position">
+                  <param name="initial_value">${initial_positions['joint_3']}</param>
+                </state_interface>
+                <!--state_interface name="velocity"/-->
+            </joint>
+            <joint name="joint_4">
+                <command_interface name="position"/>
+                <state_interface name="position">
+                  <param name="initial_value">${initial_positions['joint_4']}</param>
+                </state_interface>
+                <!--state_interface name="velocity"/-->
+            </joint>
+            <joint name="joint_5">
+                <command_interface name="position"/>
+                <state_interface name="position">
+                  <param name="initial_value">${initial_positions['joint_5']}</param>
+                </state_interface>
+                <!--state_interface name="velocity"/-->
+            </joint>
+            <joint name="joint_6">
+                <command_interface name="position"/>
+                <state_interface name="position">
+                  <param name="initial_value">${initial_positions['joint_6']}</param>
+                </state_interface>
+                <!--state_interface name="velocity"/-->
+            </joint>
+            </ros2_control>
+    </xacro:macro>
 </robot>

File: src/probot_description/urdf/probot_anno.xacro (robot description, xacro)
@@ -1,310 +1,26 @@
 <?xml version="1.0"?>
-<robot name="probot_anno" xmlns:xacro="http://ros.org/wiki/xacro">
-  <xacro:arg name="use_gazebo" default="true" />
-  <xacro:property name="M_PI" value="3.1415926536"/>
-  <link name="base_footprint"/>
-  <joint name="joint_0" type="fixed">
-    <origin xyz="0 0 0.0532" rpy="0 0 0" />
-    <parent link="base_footprint" />
-    <child link="base_link" />
-  </joint>
-  <link name="base_link">
-    <inertial>
-      <origin xyz="-0.010934 0.23134 0.0051509" rpy="0 0 0" />
-      <mass value="0.286755864167795" />
-      <inertia
-        ixx="0.000914891478336648"
-        ixy="-9.74616219194614E-08"
-        ixz="-1.22707969258407E-10"
-        iyy="0.000918304334803416"
-        iyz="-7.53317610970858E-09"
-        izz="0.00181941891671005" />
-    </inertial>
-    <visual>
-      <origin xyz="0.017266 0 0" rpy="0 0 0" />
-      <geometry>
-        <mesh filename="package://probot_description/meshes/base_link.STL" />
-      </geometry>
-      <material name="robot_color">
-        <color rgba="0.79216 0.81961 0.93333 1" />
-      </material>
-    </visual>
-    <collision>
-      <origin xyz="0.017266 0 0" rpy="0 0 0" />
-      <geometry>
-        <mesh filename="package://probot_description/meshes/base_link.STL" />
-      </geometry>
-    </collision>
-  </link>
-  <link name="link_1">
-    <inertial>
-      <origin xyz="-0.010934 0.23134 0.0051509" rpy="0 0 0" />
-      <mass value="1.50473234946919" />
-      <inertia
-        ixx="0.00667121219534555"
-        ixy="-8.54445620252032E-06"
-        ixz="1.56560865622562E-07"
-        iyy="0.00595997019373921"
-        iyz="0.000424090863023404"
-        izz="0.006430374759868" />
-    </inertial>
-    <visual>
-      <origin xyz="0 0 0" rpy="0 0 0" />
-      <geometry>
-        <mesh filename="package://probot_description/meshes/link_1.STL" />
-      </geometry>
-      <material name="robot_color">
-        <color rgba="0.79216 0.81961 0.93333 1" />
-      </material>
-    </visual>
-    <collision>
-      <origin xyz="0 0 0" rpy="0 0 0" />
-      <geometry>
-        <mesh filename="package://probot_description/meshes/link_1.STL" />
-      </geometry>
-    </collision>
-  </link>
-  <joint name="joint_1" type="revolute">
-    <origin xyz="0 0 0" rpy="1.5708 0 0" />
-    <parent link="base_link" />
-    <child link="link_1" />
-    <axis xyz="0 1 0" />
-    <limit lower="-3.1416" upper="3.1416" effort="100" velocity="3" />
-  </joint>
-  <link name="link_2">
-    <inertial>
-      <origin xyz="-0.010934 0.23134 0.0051509" rpy="0 0 0" />
-      <mass value="1.00050619907027" />
-      <inertia
-        ixx="0.0014522332353461"
-        ixy="-8.9482731163037E-06"
-        ixz="2.82386498605548E-05"
-        iyy="0.00136522040691973"
-        iyz="3.07414967244519E-06"
-        izz="0.0024851244648194" />
-    </inertial>
-    <visual>
-      <origin xyz="0 0 0" rpy="0 0 0" />
-      <geometry>
-        <mesh filename="package://probot_description/meshes/link_2.STL" />
-      </geometry>
-      <material name="robot_color">
-        <color rgba="0.79216 0.81961 0.93333 1" />
-      </material>
-    </visual>
-    <collision>
-      <origin xyz="0 0 0" rpy="0 0 0" />
-      <geometry>
-        <mesh filename="package://probot_description/meshes/link_2.STL" />
-      </geometry>
-    </collision>
-  </link>
-  <joint name="joint_2" type="revolute">
-    <origin xyz="0 0.2305 0" rpy="0 0 0" />
-    <parent link="link_1" />
-    <child link="link_2" />
-    <axis xyz="0 0 1" />
-    <limit lower="-2.0071" upper="2.0071" effort="100" velocity="3" />
-  </joint>
-  <link name="link_3">
-    <inertial>
-      <origin xyz="-0.010934 0.23134 0.0051509" rpy="0 0 0" />
-      <mass value="0.549520755006072" />
-      <inertia
-        ixx="0.000672536702276881"
-        ixy="-6.59360128441997E-06"
-        ixz="-9.19434642556495E-07"
-        iyy="0.000480817179261754"
-        iyz="4.15241325610066E-06"
-        izz="0.001032595781869" />
-    </inertial>
-    <visual>
-      <origin xyz="0 0 0" rpy="0 0 0" />
-      <geometry>
-        <mesh filename="package://probot_description/meshes/link_3.STL" />
-      </geometry>
-      <material name="robot_color">
-        <color rgba="0.79216 0.81961 0.93333 1" />
-      </material>
-    </visual>
-    <collision>
-      <origin xyz="0 0 0" rpy="0 0 0" />
-      <geometry>
-        <mesh filename="package://probot_description/meshes/link_3.STL" />
-      </geometry>
-    </collision>
-  </link>
-  <joint name="joint_3" type="revolute">
-    <origin xyz="0 0.225 0" rpy="0 0 1.5708" />
-    <parent link="link_2" />
-    <child link="link_3" />
-    <axis xyz="0 0 1" />
-    <limit lower="-2.2689" upper="2.2689" effort="100" velocity="3" />
-  </joint>
-  <link name="link_4">
-    <inertial>
-      <origin xyz="-0.010934 0.23134 0.0051509" rpy="0 0 0" />
-      <mass value="0.952497713016407" />
-      <inertia
-        ixx="0.00530614361480367"
-        ixy="7.10404845280282E-20"
-        ixz="-3.14301719378985E-20"
-        iyy="0.00354259274696511"
-        iyz="-6.5480532041068E-19"
-        izz="0.00221010202882688" />
-    </inertial>
-    <visual>
-      <origin xyz="0 0 0" rpy="0 0 0" />
-      <geometry>
-        <mesh filename="package://probot_description/meshes/link_4.STL" />
-      </geometry>
-      <material name="robot_color">
-        <color rgba="0.79216 0.81961 0.93333 1" />
-      </material>
-    </visual>
-    <collision>
-      <origin xyz="0 0 0" rpy="0 0 0" />
-      <geometry>
-        <mesh filename="package://probot_description/meshes/link_4.STL" />
-      </geometry>
-    </collision>
-  </link>
-  <joint name="joint_4" type="revolute">
-    <origin xyz="0.021 0 0.002" rpy="0 0 0" />
-    <parent link="link_3" />
-    <child link="link_4" />
-    <axis xyz="1 0 0" />
-    <limit lower="-3.1416" upper="3.1416" effort="100" velocity="3" />
-  </joint>
-  <link name="link_5">
-    <inertial>
-      <origin xyz="-0.010934 0.23134 0.0051509" rpy="0 0 0" />
-      <mass value="0.393287799668792" />
-      <inertia
-        ixx="0.000319382332386347"
-        ixy="-9.00754957688623E-10"
-        ixz="-1.75182555785641E-09"
-        iyy="0.000272873273899642"
-        iyz="-4.5738506474632E-10"
-        izz="0.000292993325719614" />
-    </inertial>
-    <visual>
-      <origin xyz="0 0 0" rpy="0 0 0" />
-      <geometry>
-        <mesh filename="package://probot_description/meshes/link_5.STL" />
-      </geometry>
-      <material name="robot_color">
-        <color rgba="0.79216 0.81961 0.93333 1" />
-      </material>
-    </visual>
-    <collision>
-      <origin xyz="0 0 0" rpy="0 0 0" />
-      <geometry>
-        <mesh filename="package://probot_description/meshes/link_5.STL" />
-      </geometry>
-    </collision>
-  </link>
-  <joint name="joint_5" type="revolute">
-    <origin xyz="0.20586 0 0" rpy="0 0 1.5708" />
-    <parent link="link_4" />
-    <child link="link_5" />
-    <axis xyz="0 0 1" />
-    <limit lower="-2.3562" upper="2.3562" effort="100" velocity="3" />
-  </joint>
-  <link name="link_6">
-    <inertial>
-      <origin xyz="-0.010934 0.23134 0.0051509" rpy="0 0 0" />
-      <mass value="0.00628105868776632" />
-      <inertia
-        ixx="5.52992389755476E-07"
-        ixy="-2.81554428275222E-22"
-        ixz="-1.40088624914581E-22"
-        iyy="5.52992389755476E-07"
-        iyz="4.83070888700992E-24"
-        izz="1.08002978042972E-06" />
-    </inertial>
-    <visual>
-      <origin xyz="0 0 0" rpy="0 0 0" />
-      <geometry>
-        <mesh filename="package://probot_description/meshes/link_6.STL" />
-      </geometry>
-      <material name="robot_color">
-        <color rgba="0.79216 0.81961 0.93333 1" />
-      </material>
-    </visual>
-    <collision>
-      <origin xyz="0 0 0" rpy="0 0 0" />
-      <geometry>
-        <mesh filename="package://probot_description/meshes/link_6.STL" />
-      </geometry>
-    </collision>
-  </link>
-  <joint name="joint_6" type="revolute">
-    <origin xyz="0 -0.042 0" rpy="0 0 0" />
-    <parent link="link_5" />
-    <child link="link_6" />
-    <axis xyz="0 -1 0" />
-    <limit lower="-3.1416" upper="3.1416" effort="100" velocity="3" />
-  </joint>
-  <link name="tool0"/>
-  <joint name="joint_tool0" type="fixed">
-    <origin xyz="0 -0.013 0" rpy="0 0 0" />
-    <parent link="link_6" />
-    <child link="tool0" />
-  </joint>
-  <!--xacro:include filename="$(find probot_description)/urdf/gripper.xacro" />
-  <xacro:probot_gripper parent="tool0">
-    <origin xyz="0 0 0" rpy="1.507 0 0" />
-  </xacro:probot_gripper-->
-  <!--xacro:if value="$(arg use_gazebo)">
+<robot xmlns:xacro="http://www.ros.org/wiki/xacro" name="probot_anno">
+    <xacro:arg name="initial_positions_file" default="$(find moveit_config)/config/initial_positions.yaml" />
+    <xacro:arg name="use_mock_hardware" default="true" />
+    <xacro:arg name="use_real_hardware" default="false" />
+    <xacro:arg name="use_gazebo" default="false" />
+    <xacro:arg name="use_isaac" default="false" />
+    <xacro:include filename="$(find probot_description)/urdf/probot_anno_macro.xacro" />
     <xacro:include filename="$(find probot_description)/urdf/probot.ros2_control.xacro" />
-    <xacro:probot_ros2_control name="GazeboSystem"/>
-  </xacro:if-->
-  <ros2_control name="ProbotRealHardware" type="system">
-    <hardware>
-      <plugin>probot_hardware/ProbotSystemHardware</plugin>
-    </hardware>
-    <joint name="joint_1">
-      <command_interface name="position"/>
-      <state_interface name="position">
-        <param name="initial_value">0.0</param>
-      </state_interface>
-      <state_interface name="velocity"/>
-    </joint>
-    <joint name="joint_2">
-      <command_interface name="position"/>
-      <state_interface name="position">
-        <param name="initial_value">0.0</param>
-      </state_interface>
-      <state_interface name="velocity"/>
-    </joint>
-    <joint name="joint_3">
-      <command_interface name="position"/>
-      <state_interface name="position">
-        <param name="initial_value">0.0</param>
-      </state_interface>
-      <state_interface name="velocity"/>
-    </joint>
-    <joint name="joint_4">
-      <command_interface name="position"/>
-      <state_interface name="position">
-        <param name="initial_value">0.0</param>
-      </state_interface>
-      <state_interface name="velocity"/>
-    </joint>
-    <joint name="joint_5">
-      <command_interface name="position"/>
-      <state_interface name="position">
-        <param name="initial_value">0.0</param>
-      </state_interface>
-      <state_interface name="velocity"/>
-    </joint>
-    <joint name="joint_6">
-      <command_interface name="position"/>
-      <state_interface name="position">
-        <param name="initial_value">0.0</param>
-      </state_interface>
-      <state_interface name="velocity"/>
-    </joint>
-  </ros2_control>
+    <xacro:probot_anno_macro />
+    <xacro:probot_anno_ros2_control
+        name="ProbotSystem"
+        initial_positions_file="$(arg initial_positions_file)"
+        use_mock_hardware="$(arg use_mock_hardware)"
+        use_real_hardware="$(arg use_real_hardware)"
+        use_gazebo="$(arg use_gazebo)"
+        use_isaac="$(arg use_isaac)"
+    />
+    <xacro:if value="$(arg use_gazebo)">
+        <gazebo>
+            <plugin filename="ign_ros2_control-system" name="ign_ros2_control::IgnitionROS2ControlPlugin">
+                <parameters>$(find moveit_config)/config/ros2_controllers.yaml</parameters>
+            </plugin>
+        </gazebo>
+    </xacro:if>
 </robot>
