Commit message: only hardware no integration

File: src/moveit_config/config/probot_anno.ros2_control.xacro (robot description, xacro)
@@ -50,5 +50,5 @@
                 <state_interface name="velocity"/>
             </joint>
-            <joint name="finger_joint1">
+            <!--joint name="finger_joint1">
                 <command_interface name="position"/>
                 <state_interface name="position">
@@ -56,5 +56,5 @@
                 </state_interface>
                 <state_interface name="velocity"/>
-            </joint>
+            </joint-->
         </ros2_control>
     </xacro:macro>

File: src/probot_description/urdf/probot.ros2_control.xacro (robot description, xacro)
@@ -36,9 +36,9 @@
         <state_interface name="velocity"/>
       </joint>
-      <joint name="finger_joint1">
+      <!--joint name="finger_joint1">
         <command_interface name="position" />
         <state_interface name="position" />
         <state_interface name="velocity" />
-      </joint>
+      </joint-->
     </ros2_control>
     <gazebo>

File: src/probot_description/urdf/probot_anno.xacro (robot description, xacro)
@@ -136,9 +136,9 @@
   </link>
   <joint name="joint_3" type="revolute">
-    <origin xyz="0 0.225 0" rpy="0 0 0" />
+    <origin xyz="0 0.225 0" rpy="0 0 1.5708" />
     <parent link="link_2" />
     <child link="link_3" />
     <axis xyz="0 0 1" />
-    <limit lower="-0.6981" upper="3.8397" effort="100" velocity="3" />
+    <limit lower="-2.2689" upper="2.2689" effort="100" velocity="3" />
   </joint>
   <link name="link_4">
@@ -206,9 +206,9 @@
   </link>
   <joint name="joint_5" type="revolute">
-    <origin xyz="0.20586 0 0" rpy="0 0 0" />
+    <origin xyz="0.20586 0 0" rpy="0 0 1.5708" />
     <parent link="link_4" />
     <child link="link_5" />
     <axis xyz="0 0 1" />
-    <limit lower="-0.7854" upper="3.9270" effort="100" velocity="3" />
+    <limit lower="-2.3562" upper="2.3562" effort="100" velocity="3" />
   </joint>
   <link name="link_6">
@@ -253,11 +253,58 @@
     <child link="tool0" />
   </joint>
-  <xacro:include filename="$(find probot_description)/urdf/gripper.xacro" />
+  <!--xacro:include filename="$(find probot_description)/urdf/gripper.xacro" />
   <xacro:probot_gripper parent="tool0">
     <origin xyz="0 0 0" rpy="1.507 0 0" />
-  </xacro:probot_gripper>
-  <xacro:if value="$(arg use_gazebo)">
+  </xacro:probot_gripper-->
+  <!--xacro:if value="$(arg use_gazebo)">
     <xacro:include filename="$(find probot_description)/urdf/probot.ros2_control.xacro" />
     <xacro:probot_ros2_control name="GazeboSystem"/>
-  </xacro:if>
+  </xacro:if-->
+  <ros2_control name="ProbotRealHardware" type="system">
+    <hardware>
+      <plugin>probot_hardware/ProbotSystemHardware</plugin>
+    </hardware>
+    <joint name="joint_1">
+      <command_interface name="position"/>
+      <state_interface name="position">
+        <param name="initial_value">0.0</param>
+      </state_interface>
+      <state_interface name="velocity"/>
+    </joint>
+    <joint name="joint_2">
+      <command_interface name="position"/>
+      <state_interface name="position">
+        <param name="initial_value">0.0</param>
+      </state_interface>
+      <state_interface name="velocity"/>
+    </joint>
+    <joint name="joint_3">
+      <command_interface name="position"/>
+      <state_interface name="position">
+        <param name="initial_value">0.0</param>
+      </state_interface>
+      <state_interface name="velocity"/>
+    </joint>
+    <joint name="joint_4">
+      <command_interface name="position"/>
+      <state_interface name="position">
+        <param name="initial_value">0.0</param>
+      </state_interface>
+      <state_interface name="velocity"/>
+    </joint>
+    <joint name="joint_5">
+      <command_interface name="position"/>
+      <state_interface name="position">
+        <param name="initial_value">0.0</param>
+      </state_interface>
+      <state_interface name="velocity"/>
+    </joint>
+    <joint name="joint_6">
+      <command_interface name="position"/>
+      <state_interface name="position">
+        <param name="initial_value">0.0</param>
+      </state_interface>
+      <state_interface name="velocity"/>
+    </joint>
+  </ros2_control>
 </robot>

Commit message: add gripper

File: src/moveit_config/config/probot_anno.ros2_control.xacro (robot description, xacro)
@@ -50,11 +50,11 @@
                 <state_interface name="velocity"/>
             </joint>
-            <!--joint name="finger_joint1">
+            <joint name="Active_Gear_Joint">
                 <command_interface name="position"/>
                 <state_interface name="position">
-                  <param name="initial_value">${initial_positions['finger_joint1']}</param>
+                  <param name="initial_value">${initial_positions['Active_Gear_Joint']}</param>
                 </state_interface>
                 <state_interface name="velocity"/>
-            </joint-->
+            </joint>
         </ros2_control>
     </xacro:macro>

File: src/probot_description/urdf/probot.ros2_control.xacro (robot description, xacro)
@@ -60,4 +60,14 @@
                 <!--state_interface name="velocity"/-->
             </joint>
+            <joint name="Active_Gear_Joint">
+                <command_interface name="position"/>
+                <state_interface name="position">
+                  <param name="initial_value">${initial_positions['Active_Gear_Joint']}</param>
+                </state_interface>
+            </joint>
+            <gpio name="iris_shutter">
+                <command_interface name="state"/>
+                <state_interface name="state"/>
+            </gpio>
             </ros2_control>
     </xacro:macro>

File: src/probot_description/urdf/probot_anno.xacro (robot description, xacro)
@@ -7,6 +7,8 @@
     <xacro:arg name="use_isaac" default="false" />
     <xacro:include filename="$(find probot_description)/urdf/probot_anno_macro.xacro" />
+    <xacro:include filename="$(find probot_description)/urdf/gripper_macro.xacro" />
     <xacro:include filename="$(find probot_description)/urdf/probot.ros2_control.xacro" />
     <xacro:probot_anno_macro />
+    <xacro:probot_gripper parent="link_6" />
     <xacro:probot_anno_ros2_control
         name="ProbotSystem"

File: src/probot_description/urdf/probot_anno_macro.xacro (robot description, xacro)
@@ -219,10 +219,10 @@
       <limit lower="-3.1416" upper="3.1416" effort="100" velocity="3" />
     </joint>
-    <link name="tool0"/>
+    <!--link name="tool0"/>
     <joint name="joint_tool0" type="fixed">
       <origin xyz="0 -0.013 0" rpy="0 0 0" />
       <parent link="link_6" />
       <child link="tool0" />
-    </joint>
+    </joint-->
     </xacro:macro>
 </robot>

Commit message: gripper urdf modifications

File: src/moveit_config/config/probot_anno.ros2_control.xacro (robot description, xacro)
@@ -57,4 +57,11 @@
                 <state_interface name="velocity"/>
             </joint>
+            <joint name="Door_Joint">
+                <command_interface name="position"/>
+                <state_interface name="position">
+                  <param name="initial_value">${initial_positions['Door_Joint']}</param>
+                </state_interface>
+                <state_interface name="velocity"/>
+            </joint>
         </ros2_control>
     </xacro:macro>

File: src/probot_description/urdf/probot.ros2_control.xacro (robot description, xacro)
@@ -66,4 +66,10 @@
                 </state_interface>
             </joint>
+            <joint name="Door_Joint">
+                <command_interface name="position"/>
+                <state_interface name="position">
+                  <param name="initial_value">${initial_positions['Door_Joint']}</param>
+                </state_interface>
+            </joint>
             <xacro:if value="${use_gazebo}">
                 <joint name="Passive_Gear_Joint">

File: src/probot_description/urdf/probot_anno.xacro (robot description, xacro)
@@ -7,5 +7,5 @@
     <xacro:arg name="use_isaac" default="false" />
     <xacro:include filename="$(find probot_description)/urdf/probot_anno_macro.xacro" />
-    <xacro:include filename="$(find probot_description)/urdf/gripper_macro.xacro" />
+    <xacro:include filename="$(find probot_description)/urdf/new_gripper_macro.xacro" />
     <xacro:include filename="$(find probot_description)/urdf/probot.ros2_control.xacro" />
     <xacro:probot_anno_macro />

Commit message: new urdf with iris

File: src/moveit_config/config/probot_anno.ros2_control.xacro (robot description, xacro)
@@ -2,5 +2,5 @@
 <robot xmlns:xacro="http://www.ros.org/wiki/xacro">
     <xacro:macro name="probot_anno_ros2_control" params="name initial_positions_file">
-        <xacro:property name="initial_positions" value="${load_yaml(initial_positions_file)['initial_positions']}"/>
+        <xacro:property name="initial_positions" value="${xacro.load_yaml(initial_positions_file)['initial_positions']}"/>
         <ros2_control name="${name}" type="system">
             <hardware>
@@ -50,8 +50,15 @@
                 <state_interface name="velocity"/>
             </joint>
-            <joint name="Active_Gear_Joint">
+            <joint name="Active_Scissors_Gear_Joint">
                 <command_interface name="position"/>
                 <state_interface name="position">
-                  <param name="initial_value">${initial_positions['Active_Gear_Joint']}</param>
+                  <param name="initial_value">${initial_positions['Active_Scissors_Gear_Joint']}</param>
+                </state_interface>
+                <state_interface name="velocity"/>
+            </joint>
+            <joint name="Iris_Active_Gear_Joint">
+                <command_interface name="position"/>
+                <state_interface name="position">
+                  <param name="initial_value">${initial_positions['Iris_Active_Gear_Joint']}</param>
                 </state_interface>
                 <state_interface name="velocity"/>

File: src/probot_description/urdf/probot.ros2_control.xacro (robot description, xacro)
@@ -2,5 +2,5 @@
 <robot xmlns:xacro="http://www.ros.org/wiki/xacro">
     <xacro:macro name="probot_anno_ros2_control" params="name initial_positions_file use_mock_hardware use_real_hardware use_gazebo use_isaac">
-        <xacro:property name="initial_positions" value="${load_yaml(initial_positions_file)['initial_positions']}"/>
+        <xacro:property name="initial_positions" value="${xacro.load_yaml(initial_positions_file)['initial_positions']}"/>
         <ros2_control name="${name}" type="system">
             <hardware>
@@ -23,5 +23,4 @@
                   <param name="initial_value">${initial_positions['joint_1']}</param>
                 </state_interface>
-                <!--state_interface name="velocity"/-->
             </joint>
             <joint name="joint_2">
@@ -30,5 +29,4 @@
                   <param name="initial_value">${initial_positions['joint_2']}</param>
                 </state_interface>
-                <!--state_interface name="velocity"/-->
             </joint>
             <joint name="joint_3">
@@ -37,5 +35,4 @@
                   <param name="initial_value">${initial_positions['joint_3']}</param>
                 </state_interface>
-                <!--state_interface name="velocity"/-->
             </joint>
             <joint name="joint_4">
@@ -44,5 +41,4 @@
                   <param name="initial_value">${initial_positions['joint_4']}</param>
                 </state_interface>
-                <!--state_interface name="velocity"/-->
             </joint>
             <joint name="joint_5">
@@ -51,5 +47,4 @@
                   <param name="initial_value">${initial_positions['joint_5']}</param>
                 </state_interface>
-                <!--state_interface name="velocity"/-->
             </joint>
             <joint name="joint_6">
@@ -58,10 +53,9 @@
                   <param name="initial_value">${initial_positions['joint_6']}</param>
                 </state_interface>
-                <!--state_interface name="velocity"/-->
             </joint>
-            <joint name="Active_Gear_Joint">
+            <joint name="Active_Scissors_Gear_Joint">
                 <command_interface name="position"/>
                 <state_interface name="position">
-                  <param name="initial_value">${initial_positions['Active_Gear_Joint']}</param>
+                  <param name="initial_value">${initial_positions['Active_Scissors_Gear_Joint']}</param>
                 </state_interface>
             </joint>
@@ -72,16 +66,55 @@
                 </state_interface>
             </joint>
+            <joint name="Iris_Active_Gear_Joint">
+                <command_interface name="position"/>
+                <state_interface name="position">
+                  <param name="initial_value">${initial_positions['Iris_Active_Gear_Joint']}</param>
+                </state_interface>
+            </joint>
             <xacro:if value="${use_gazebo}">
+                <!-- Passive Scissors mimics Active Scissors -->
                 <joint name="Passive_Scissors_Gear_Joint">
-                    <param name="mimic">Active_Gear_Joint</param>
+                    <param name="mimic">Active_Scissors_Gear_Joint</param>
                     <param name="multiplier">-1.0</param>
-                    <state_interface name="position"/>
+                    <command_interface name="position"/>
+                    <state_interface name="position">
+                        <param name="initial_value">0.0</param>
+                    </state_interface>
                 </joint>
+                <!-- Passive Iris Gear mimics Active Iris Gear -->
+                <joint name="Iris_Passive_Gear_Joint">
+                    <param name="mimic">Iris_Active_Gear_Joint</param>
+                    <param name="multiplier">-0.3367</param>
+                    <command_interface name="position"/>
+                    <state_interface name="position">
+                        <param name="initial_value">0.0</param>
+                    </state_interface>
+                </joint>
+                <!-- ALL 12 Blades mimic the Active Iris Gear DIRECTLY to avoid chain-mimic bugs -->
+                <!-- Multiplier = -0.3367 (passive gear) * 1.6 (blade to passive gear) = -0.53872 -->
+                <xacro:macro name="mimic_iris" params="num">
+                    <joint name="Iris${num}_Joint">
+                        <param name="mimic">Iris_Active_Gear_Joint</param>
+                        <param name="multiplier">-0.53872</param>
+                        <command_interface name="position"/>
+                        <state_interface name="position">
+                            <param name="initial_value">0.0</param>
+                        </state_interface>
+                    </joint>
+                </xacro:macro>
+                <xacro:mimic_iris num="1"/>
+                <xacro:mimic_iris num="2"/>
+                <xacro:mimic_iris num="3"/>
+                <xacro:mimic_iris num="4"/>
+                <xacro:mimic_iris num="5"/>
+                <xacro:mimic_iris num="6"/>
+                <xacro:mimic_iris num="7"/>
+                <xacro:mimic_iris num="8"/>
+                <xacro:mimic_iris num="9"/>
+                <xacro:mimic_iris num="10"/>
+                <xacro:mimic_iris num="11"/>
+                <xacro:mimic_iris num="12"/>
             </xacro:if>
-            <gpio name="iris_shutter">
-                <command_interface name="state"/>
-                <state_interface name="state"/>
-            </gpio>
-            </ros2_control>
+        </ros2_control>
     </xacro:macro>
 </robot>

File: src/probot_description/urdf/probot_anno.xacro (robot description, xacro)
@@ -7,5 +7,5 @@
     <xacro:arg name="use_isaac" default="false" />
     <xacro:include filename="$(find probot_description)/urdf/probot_anno_macro.xacro" />
-    <xacro:include filename="$(find probot_description)/urdf/new_gripper_macro.xacro" />
+    <xacro:include filename="$(find probot_description)/urdf/gripper_macro.xacro" />
     <xacro:include filename="$(find probot_description)/urdf/probot.ros2_control.xacro" />
     <xacro:probot_anno_macro />

File: src/probot_description/urdf/probot_anno_macro.xacro (robot description, xacro)
@@ -3,8 +3,67 @@
   <xacro:macro name="probot_anno_macro">
     <xacro:property name="M_PI" value="3.1415926536"/>
+    <!-- Materials -->
+    <material name="offwhite">
+      <color rgba="0.95 0.95 0.92 1" />
+    </material>
+    <material name="kinect_dark">
+      <color rgba="0.15 0.15 0.15 1" /> <!-- The classic dark matte grey of the Kinect -->
+    </material>
+    <!-- Fix robot to world -->
     <link name="world"/>
+    <joint name="world_to_robot_base" type="fixed">
+      <origin xyz="0 0 0" rpy="0 0 0" />
+      <parent link="world" />
+      <child link="robot_base" />
+    </joint>
+    <!-- New Robot Base -->
+    <link name="robot_base">
+      <inertial>
+        <origin xyz="-0.26475 0.051293 0.019346" rpy="0 0 0" />
+        <mass value="1.4191" />
+        <inertia ixx="0.012341" ixy="0.0054099" ixz="0.0023347" iyy="0.03677" iyz="-0.0018374" izz="0.047034" />
+      </inertial>
+      <visual>
+        <origin xyz="0 0 0" rpy="0 0 0" />
+        <geometry>
+          <mesh filename="package://probot_description/meshes/robot_base.STL" />
+        </geometry>
+      <material name="kinect_dark" />
+      </visual>
+      <collision>
+        <origin xyz="0 0 0" rpy="0 0 0" />
+        <geometry>
+          <mesh filename="package://probot_description/meshes/robot_base.STL" />
+        </geometry>
+      </collision>
+    </link>
+    <!-- Kinect optical frames -->
+    <link name="camera_link1"/>
+    <joint name="camera_joint1" type="fixed">
+      <origin xyz="-0.27393 0.13681 0.05339" rpy="-1.509 0 0" />
+      <parent link="robot_base" />
+      <child link="camera_link1" />
+    </joint>
+    <link name="camera_link2"/>
+    <joint name="camera_joint2" type="fixed">
+      <origin xyz="-0.32393 0.13681 0.05339" rpy="-1.509 0 0" />
+      <parent link="robot_base" />
+      <child link="camera_link2" />
+    </joint>
+    <link name="camera_link3"/>
+    <joint name="camera_joint3" type="fixed">
+      <origin xyz="-0.34993 0.13681 0.05339" rpy="-1.509 0 0" />
+      <parent link="robot_base" />
+      <child link="camera_link3" />
+    </joint>
+    <link name="base_footprint"/>
+    <joint name="robot_base_to_base_footprint" type="fixed">
+      <origin xyz="0 0 -0.017" rpy="0 0 0"/>
+      <parent link="robot_base"/>
+      <child link="base_footprint"/>
+    </joint>
     <joint name="joint_0" type="fixed">
       <origin xyz="0 0 0.0532" rpy="0 0 0" />
-      <parent link="world" />
+      <parent link="base_footprint" />
       <child link="base_link" />
     </joint>
@@ -20,14 +79,12 @@
         <origin xyz="0.017266 0 0" rpy="0 0 0" />
         <geometry>
-          <mesh filename="package://probot_description/meshes/base_link.STL" />
-        </geometry>
-        <material name="robot_color">
-          <color rgba="0.79216 0.81961 0.93333 1" />
-        </material>
+          <mesh filename="package://probot_description/meshes/new_base_link.stl" />
+        </geometry>
+      <material name="offwhite" />
       </visual>
       <collision>
         <origin xyz="0.017266 0 0" rpy="0 0 0" />
         <geometry>
-          <mesh filename="package://probot_description/meshes/base_link.STL" />
+          <mesh filename="package://probot_description/meshes/new_base_link.stl" />
         </geometry>
       </collision>
@@ -46,7 +103,5 @@
           <mesh filename="package://probot_description/meshes/link_1.STL" />
         </geometry>
-        <material name="robot_color">
-          <color rgba="0.79216 0.81961 0.93333 1" />
-        </material>
+        <material name="offwhite" />
       </visual>
       <collision>
@@ -77,7 +132,5 @@
           <mesh filename="package://probot_description/meshes/link_2.STL" />
         </geometry>
-        <material name="robot_color">
-          <color rgba="0.79216 0.81961 0.93333 1" />
-        </material>
+        <material name="offwhite" />
       </visual>
       <collision>
@@ -108,7 +161,5 @@
           <mesh filename="package://probot_description/meshes/link_3.STL" />
         </geometry>
-        <material name="robot_color">
-          <color rgba="0.79216 0.81961 0.93333 1" />
-        </material>
+        <material name="offwhite" />
       </visual>
       <collision>
@@ -139,7 +190,5 @@
           <mesh filename="package://probot_description/meshes/link_4.STL" />
         </geometry>
-        <material name="robot_color">
-          <color rgba="0.79216 0.81961 0.93333 1" />
-        </material>
+        <material name="offwhite" />
       </visual>
       <collision>
@@ -170,7 +219,5 @@
           <mesh filename="package://probot_description/meshes/link_5.STL" />
         </geometry>
-        <material name="robot_color">
-          <color rgba="0.79216 0.81961 0.93333 1" />
-        </material>
+        <material name="offwhite" />
       </visual>
       <collision>
@@ -201,7 +248,5 @@
           <mesh filename="package://probot_description/meshes/link_6.STL" />
         </geometry>
-        <material name="robot_color">
-          <color rgba="0.79216 0.81961 0.93333 1" />
-        </material>
+        <material name="offwhite" />
       </visual>
       <collision>
